Commit message: Unified style and namings

File: pmb2_description/ros2_control/ros2_control.urdf.xacro (robot description, xacro)
@@ -15,5 +15,5 @@
   <!-- INCLUDES -->
   <xacro:include filename="$(find pmb2_description)/urdf/wheels/wheel.ros2_control.xacro"/>
-  <xacro:include filename="$(find pmb2_description)/urdf/sensors/sensors.ros2_control.xacro"/>
+  <xacro:include filename="$(find pmb2_description)/urdf/sensors/imu.ros2_control.xacro"/>
   <!-- MACRO DEFINITION-->
   <xacro:macro name="pmb2_ros2_control">

File: pmb2_description/urdf/cameras_add_on/cameras_add_on.urdf.xacro (robot description, xacro)
@@ -1,6 +1,20 @@
 <?xml version="1.0"?>
+<!--
+  Copyright (c) 2024 PAL Robotics S.L. All rights reserved.
+  Licensed under the Apache License, Version 2.0 (the "License");
+  you may not use this file except in compliance with the License.
+  You may obtain a copy of the License at
+      http://www.apache.org/licenses/LICENSE-2.0
+  Unless required by applicable law or agreed to in writing, software
+  distributed under the License is distributed on an "AS IS" BASIS,
+  WITHOUT WARRANTIES OR CONDITIONS OF ANY KIND, either express or implied.
+  See the License for the specific language governing permissions and
+  limitations under the License.
+-->
 <robot xmlns:xacro="http://ros.org/wiki/xacro">
-  <!--File includes-->
+  <!-- INCLUDES -->
   <xacro:include filename="$(find pal_urdf_utils)/urdf/deg_to_rad.urdf.xacro" />
+  <xacro:include filename="$(find pmb2_description)/urdf/sensors/courier.urdf.xacro" />
+  <!-- MACRO DEFINITION-->
   <xacro:macro name="cameras_add_on" params="name parent">
     <link name="${name}_link">
@@ -32,4 +46,3 @@
     </joint>
   </xacro:macro>
-  <xacro:include filename="$(find pmb2_description)/urdf/sensors/courier.urdf.xacro" />
 </robot>

File: pmb2_description/urdf/dock/dock.urdf.xacro (robot description, xacro)
@@ -1,5 +1,5 @@
 <?xml version="1.0"?>
 <!--
-  Copyright (c) 2022 PAL Robotics S.L. All rights reserved.
+  Copyright (c) 2024 PAL Robotics S.L. All rights reserved.
   Licensed under the Apache License, Version 2.0 (the "License");
   you may not use this file except in compliance with the License.
@@ -11,8 +11,10 @@
   See the License for the specific language governing permissions and
   limitations under the License.
- -->
+-->
 <robot xmlns:xacro="http://ros.org/wiki/xacro">
+  <!-- INCLUDES -->
   <xacro:include filename="$(find pal_urdf_utils)/urdf/deg_to_rad.urdf.xacro"/>
   <xacro:include filename="$(find pmb2_description)/urdf/sensors/ir_emitter.urdf.xacro"/>
+  <!-- MACRO DEFINITION -->
   <xacro:macro name="dock" params="name">
     <!-- Dock -->
@@ -27,5 +29,4 @@
         <geometry>
           <mesh filename="package://pmb2_description/meshes/dock/dock.stl" />
-          <!--mesh filename="package://pmb2_description/meshes/dock/dock.dae" /-->
         </geometry>
         <material name="LightGrey" />

File: pmb2_description/urdf/sensors/bumper.urdf.xacro (robot description, xacro)
@@ -19,7 +19,5 @@
         <origin xyz="-0.05002000000 0.00000000000 0.00000000000" rpy="0 0 0"/>
         <mass value="0.15368000000"/>
-        <inertia ixx="0.00281031560" ixy="0.00000000000" ixz="0.00000000000"
-                 iyy="0.00021829037" iyz="0.00000000000"
-                 izz="0.00302258512"/>
+        <inertia ixx="0.00281031560" ixy="0.00000000000" ixz="0.00000000000" iyy="0.00021829037" iyz="0.00000000000" izz="0.00302258512"/>
       </inertial>
       <visual>
@@ -42,5 +40,5 @@
       <xacro:insert_block name="origin"/>
       <parent link="${parent}_link"/>
-      <child  link="${name}_link"/>
+      <child link="${name}_link"/>
     </joint>
     <!-- gazebo extensions -->

File: pmb2_description/urdf/sensors/courier.urdf.xacro (robot description, xacro)
@@ -39,46 +39,34 @@
   <xacro:structure_sensor name="base_rgbd_camera" parent="base">
     <!-- Pose of sensor frame wrt to base -->
-    <origin
-      xyz="${base_rgbd_x} ${base_rgbd_y} ${base_rgbd_z}"
-      rpy="${base_rgbd_R * deg_to_rad} ${base_rgbd_P * deg_to_rad} ${base_rgbd_Y * deg_to_rad}"/>
+    <origin xyz="${base_rgbd_x} ${base_rgbd_y} ${base_rgbd_z}" rpy="${base_rgbd_R * deg_to_rad} ${base_rgbd_P * deg_to_rad} ${base_rgbd_Y * deg_to_rad}"/>
     <!-- Pose of optical frame wrt to sensor -->
-    <origin
-      xyz="0 0 0"
-      rpy="${-90 * deg_to_rad} 0 ${-90 * deg_to_rad}"/>
+    <origin xyz="0 0 0" rpy="${-90 * deg_to_rad} 0 ${-90 * deg_to_rad}"/>
   </xacro:structure_sensor>
   <!-- RGBD roof -->
   <xacro:structure_sensor name="roof_rgbd_camera" parent="base">
     <!-- Pose of sensor frame wrt to base -->
-    <origin
-      xyz="${roof_rgbd_x} ${roof_rgbd_y} ${roof_rgbd_z}"
-      rpy="${roof_rgbd_R * deg_to_rad} ${roof_rgbd_P * deg_to_rad} ${roof_rgbd_Y * deg_to_rad}"/>
+    <origin xyz="${roof_rgbd_x} ${roof_rgbd_y} ${roof_rgbd_z}" rpy="${roof_rgbd_R * deg_to_rad} ${roof_rgbd_P * deg_to_rad} ${roof_rgbd_Y * deg_to_rad}"/>
     <!-- Pose of optical frame wrt to sensor -->
-    <origin
-      xyz="0 0 0"
-      rpy="${-90 * deg_to_rad} 0 ${-90 * deg_to_rad}"/>
+    <origin xyz="0 0 0" rpy="${-90 * deg_to_rad} 0 ${-90 * deg_to_rad}"/>
   </xacro:structure_sensor>
   <!-- RGB -->
   <xacro:elp_rgb name="rgb_camera" parent="base">
     <!-- Pose of sensor frame wrt to base -->
-    <origin
-      xyz="${rgb_x} ${rgb_y} ${rgb_z}"
-      rpy="${rgb_R * deg_to_rad} ${rgb_P * deg_to_rad} ${rgb_Y * deg_to_rad}"/>
+    <origin xyz="${rgb_x} ${rgb_y} ${rgb_z}" rpy="${rgb_R * deg_to_rad} ${rgb_P * deg_to_rad} ${rgb_Y * deg_to_rad}"/>
     <!-- Pose of optical frame wrt to sensor -->
-    <origin
-      xyz="0 0 0"
-      rpy="${-90 * deg_to_rad} 0 ${-90 * deg_to_rad}"/>
+    <origin xyz="0 0 0" rpy="${-90 * deg_to_rad} 0 ${-90 * deg_to_rad}"/>
   </xacro:elp_rgb>
   <!-- RGBD Laser Link -->
   <joint name="rgbd_laser_joint" type="fixed">
-      <parent link="base_footprint"/>
-      <child link="rgbd_laser_link"/>
-      <origin xyz="-0.9 0 0" rpy="0 0 0" />
+    <parent link="base_footprint"/>
+    <child link="rgbd_laser_link"/>
+    <origin xyz="-0.9 0 0" rpy="0 0 0" />
   </joint>
   <link name="rgbd_laser_link">
-      <inertial>
-          <origin xyz="0 0 0" rpy="0 0 0"/>
-          <mass value="0.0001" />
-          <inertia ixx="0.0001"  ixy="0"  ixz="0" iyy="0.0001" iyz="0" izz="0.0001" />
-      </inertial>
+    <inertial>
+      <origin xyz="0 0 0" rpy="0 0 0"/>
+      <mass value="0.0001" />
+      <inertia ixx="0.0001" ixy="0" ixz="0" iyy="0.0001" iyz="0" izz="0.0001" />
+    </inertial>
   </link>
 </robot>

File: pmb2_description/urdf/sensors/elp_rgb.urdf.xacro (robot description, xacro)
@@ -13,5 +13,5 @@
  -->
 <robot xmlns:xacro="http://ros.org/wiki/xacro">
- <xacro:include filename="$(find pmb2_description)/urdf/sensors/elp_rgb.gazebo.xacro" />
+  <xacro:include filename="$(find pmb2_description)/urdf/sensors/elp_rgb.gazebo.xacro" />
   <!-- Macro -->
   <xacro:macro name="elp_rgb" params="name parent *origin *optical_origin">
@@ -27,7 +27,5 @@
         <origin xyz="0 0 0" rpy="0 0 0"/>
         <mass value="0.01" />
-        <inertia ixx="0.000030"  ixy="0.0"  ixz="0.0"
-                 iyy="0.000030"  iyz="0.0"
-                 izz="0.000002" />
+        <inertia ixx="0.000030" ixy="0.0" ixz="0.0" iyy="0.000030" iyz="0.0" izz="0.000002" />
       </inertial>
       <visual>

File: pmb2_description/urdf/sensors/hokuyo_urg_04lx_ug01_laser.gazebo.xacro (robot description, xacro)
@@ -24,5 +24,5 @@
               <!-- 683 steps in 240deg fov -->
               <samples>${683*(max_angle - min_angle)/(240.0 * deg_to_rad)}</samples>
-              <resolution>1</resolution> <!-- not the sensor resolution; just 1 -->
+              <resolution>1</resolution>              <!-- not the sensor resolution; just 1 -->
               <min_angle>${min_angle}</min_angle>
               <max_angle>${max_angle}</max_angle>
@@ -40,10 +40,10 @@
           </noise>
         </ray>
-      	<plugin name="${name}" filename="libgazebo_ros_ray_sensor.so">
+        <plugin name="${name}" filename="libgazebo_ros_ray_sensor.so">
           <ros>
-      	    <remapping>~/out:=${ros_topic}</remapping>
+            <remapping>~/out:=${ros_topic}</remapping>
           </ros>
           <output_type>sensor_msgs/LaserScan</output_type>
-      	  <frame_name>${name}_link</frame_name>
+          <frame_name>${name}_link</frame_name>
         </plugin>
       </sensor>

File: pmb2_description/urdf/sensors/hokuyo_urg_04lx_ug01_laser.urdf.xacro (robot description, xacro)
@@ -19,7 +19,5 @@
         <origin xyz="0 0 -0.04480000000" rpy="0 0 0"/>
         <mass value="0.22963000000"/>
-        <inertia ixx="0.00003393164" ixy="0.00000064943" ixz="0.00000000000"
-                 iyy="0.00001849658" iyz="0.00000000000"
-                 izz="0.00005027615"/>
+        <inertia ixx="0.00003393164" ixy="0.00000064943" ixz="0.00000000000" iyy="0.00001849658" iyz="0.00000000000" izz="0.00005027615"/>
       </inertial>
       <visual>
@@ -35,5 +33,5 @@
       <xacro:insert_block name="origin"/>
       <parent link="${parent}_link"/>
-      <child  link="${name}_link"/>
+      <child link="${name}_link"/>
     </joint>
     <!-- gazebo extensions -->

File: pmb2_description/urdf/sensors/range.gazebo.xacro (robot description, xacro)
@@ -13,5 +13,5 @@
  -->
 <robot xmlns:xacro="http://ros.org/wiki/xacro">
-  <xacro:macro name="range_gazebo" params="name ros_topic update_rate maxRange minRange fov radiation" >
+  <xacro:macro name="range_gazebo" params="name ros_topic update_rate maxRange minRange fov radiation">
     <gazebo reference="${name}_link">
       <sensor type="ray" name="${name}">
@@ -39,5 +39,5 @@
             <resolution>0.01</resolution>
           </range>
-	  <noise>
+          <noise>
             <type>gaussian</type>
             <mean>0.0</mean>
@@ -45,12 +45,12 @@
           </noise>
         </ray>
-	<plugin name="${name}_gazebo_ros_range" filename="libgazebo_ros_ray_sensor.so">
-            <ros>
-                <namespace></namespace>
-                <remapping>~/out:=${ros_topic}</remapping>
-            </ros>
-            <output_type>sensor_msgs/Range</output_type>
-	    <radiation_type>${radiation}</radiation_type>
-            <frame_name>${name}_link</frame_name>
+        <plugin name="${name}_gazebo_ros_range" filename="libgazebo_ros_ray_sensor.so">
+          <ros>
+            <namespace></namespace>
+            <remapping>~/out:=${ros_topic}</remapping>
+          </ros>
+          <output_type>sensor_msgs/Range</output_type>
+          <radiation_type>${radiation}</radiation_type>
+          <frame_name>${name}_link</frame_name>
         </plugin>
       </sensor>

File: pmb2_description/urdf/sensors/range.urdf.xacro (robot description, xacro)
@@ -19,7 +19,5 @@
         <origin xyz="0 0 0" rpy="0 0 0"/>
         <mass value="0.001"/>
-        <inertia ixx="0.000001" ixy="0" ixz="0"
-                 iyy="0.000001" iyz="0"
-                 izz="0.000001"/>
+        <inertia ixx="0.000001" ixy="0" ixz="0" iyy="0.000001" iyz="0" izz="0.000001"/>
       </inertial>
       <visual>

File: pmb2_description/urdf/sensors/sick_tim551_laser.gazebo.xacro (robot description, xacro)
@@ -24,5 +24,5 @@
               <!-- 270 steps in 270deg fov -->
               <samples>${270*(max_angle - min_angle)/(270.0 * deg_to_rad)}</samples>
-              <resolution>1</resolution> <!-- not the sensor resolution; just 1 -->
+              <resolution>1</resolution>              <!-- not the sensor resolution; just 1 -->
               <min_angle>${min_angle}</min_angle>
               <max_angle>${max_angle}</max_angle>
@@ -40,10 +40,10 @@
           </noise>
         </ray>
-      	<plugin name="${name}" filename="libgazebo_ros_ray_sensor.so">
+        <plugin name="${name}" filename="libgazebo_ros_ray_sensor.so">
           <ros>
-      	    <remapping>~/out:=${ros_topic}</remapping>
+            <remapping>~/out:=${ros_topic}</remapping>
           </ros>
           <output_type>sensor_msgs/LaserScan</output_type>
-      	  <frame_name>${name}_link</frame_name>
+          <frame_name>${name}_link</frame_name>
         </plugin>
       </sensor>

File: pmb2_description/urdf/sensors/sick_tim551_laser.urdf.xacro (robot description, xacro)
@@ -15,11 +15,9 @@
   <xacro:include filename="$(find pmb2_description)/urdf/sensors/sick_tim551_laser.gazebo.xacro" />
   <xacro:macro name="sick_tim551_laser" params="name parent *origin ros_topic update_rate min_angle max_angle">
-     <link name="${name}_link" type="laser">
+    <link name="${name}_link" type="laser">
       <inertial>
         <origin xyz="-0.02559000000 -0.00056000000 -0.05732000000" rpy="0 0 0"/>
         <mass value="0.28922000000"/>
-        <inertia ixx="0.00002628919" ixy="0.00000024298" ixz="-0.00000368129"
-                 iyy="0.00003374542" iyz="-0.00000001330"
-                 izz="0.00005832599"/>
+        <inertia ixx="0.00002628919" ixy="0.00000024298" ixz="-0.00000368129" iyy="0.00003374542" iyz="-0.00000001330" izz="0.00005832599"/>
       </inertial>
       <visual>
@@ -35,5 +33,5 @@
       <xacro:insert_block name="origin"/>
       <parent link="${parent}_link"/>
-      <child  link="${name}_link"/>
+      <child link="${name}_link"/>
     </joint>
     <!-- gazebo extensions -->

File: pmb2_description/urdf/sensors/sick_tim561_laser.gazebo.xacro (robot description, xacro)
@@ -24,5 +24,5 @@
               <!-- 818 (270/0.33) steps in 270deg fov -->
               <samples>${818*(max_angle - min_angle)/(270.0 * deg_to_rad)}</samples>
-              <resolution>1</resolution> <!-- not the sensor resolution; just 1 -->
+              <resolution>1</resolution>              <!-- not the sensor resolution; just 1 -->
               <min_angle>${min_angle}</min_angle>
               <max_angle>${max_angle}</max_angle>
@@ -40,10 +40,10 @@
           </noise>
         </ray>
-      	<plugin name="${name}" filename="libgazebo_ros_ray_sensor.so">
+        <plugin name="${name}" filename="libgazebo_ros_ray_sensor.so">
           <ros>
-      	    <remapping>~/out:=${ros_topic}</remapping>
+            <remapping>~/out:=${ros_topic}</remapping>
           </ros>
           <output_type>sensor_msgs/LaserScan</output_type>
-      	  <frame_name>${name}_link</frame_name>
+          <frame_name>${name}_link</frame_name>
         </plugin>
       </sensor>

File: pmb2_description/urdf/sensors/sick_tim561_laser.urdf.xacro (robot description, xacro)
@@ -15,11 +15,9 @@
   <xacro:include filename="$(find pmb2_description)/urdf/sensors/sick_tim561_laser.gazebo.xacro" />
   <xacro:macro name="sick_tim561_laser" params="name parent *origin ros_topic update_rate min_angle max_angle">
-     <link name="${name}_link" type="laser">
+    <link name="${name}_link" type="laser">
       <inertial>
         <origin xyz="-0.02559000000 -0.00056000000 -0.05732000000" rpy="0 0 0"/>
         <mass value="0.28922000000"/>
-        <inertia ixx="0.00002628919" ixy="0.00000024298" ixz="-0.00000368129"
-                 iyy="0.00003374542" iyz="-0.00000001330"
-                 izz="0.00005832599"/>
+        <inertia ixx="0.00002628919" ixy="0.00000024298" ixz="-0.00000368129" iyy="0.00003374542" iyz="-0.00000001330" izz="0.00005832599"/>
       </inertial>
       <visual>
@@ -35,5 +33,5 @@
       <xacro:insert_block name="origin"/>
       <parent link="${parent}_link"/>
-      <child  link="${name}_link"/>
+      <child link="${name}_link"/>
     </joint>
     <!-- gazebo extensions -->

File: pmb2_description/urdf/sensors/sick_tim571_laser.gazebo.xacro (robot description, xacro)
@@ -24,5 +24,5 @@
               <!-- 818 (270/0.33) steps in 270deg fov -->
               <samples>${818*(max_angle - min_angle)/(270.0 * deg_to_rad)}</samples>
-              <resolution>1</resolution> <!-- not the sensor resolution; just 1 -->
+              <resolution>1</resolution>              <!-- not the sensor resolution; just 1 -->
               <min_angle>${min_angle}</min_angle>
               <max_angle>${max_angle}</max_angle>
@@ -40,10 +40,10 @@
           </noise>
         </ray>
-      	<plugin name="${name}" filename="libgazebo_ros_ray_sensor.so">
+        <plugin name="${name}" filename="libgazebo_ros_ray_sensor.so">
           <ros>
-      	    <remapping>~/out:=${ros_topic}</remapping>
+            <remapping>~/out:=${ros_topic}</remapping>
           </ros>
           <output_type>sensor_msgs/LaserScan</output_type>
-      	  <frame_name>${name}_link</frame_name>
+          <frame_name>${name}_link</frame_name>
         </plugin>
       </sensor>

File: pmb2_description/urdf/sensors/sick_tim571_laser.urdf.xacro (robot description, xacro)
@@ -15,11 +15,9 @@
   <xacro:include filename="$(find pmb2_description)/urdf/sensors/sick_tim571_laser.gazebo.xacro" />
   <xacro:macro name="sick_tim571_laser" params="name parent *origin ros_topic update_rate min_angle max_angle">
-     <link name="${name}_link" type="laser">
+    <link name="${name}_link" type="laser">
       <inertial>
         <origin xyz="-0.02559000000 -0.00056000000 -0.05732000000" rpy="0 0 0"/>
         <mass value="0.28922000000"/>
-        <inertia ixx="0.00002628919" ixy="0.00000024298" ixz="-0.00000368129"
-                 iyy="0.00003374542" iyz="-0.00000001330"
-                 izz="0.00005832599"/>
+        <inertia ixx="0.00002628919" ixy="0.00000024298" ixz="-0.00000368129" iyy="0.00003374542" iyz="-0.00000001330" izz="0.00005832599"/>
       </inertial>
       <visual>
@@ -35,5 +33,5 @@
       <xacro:insert_block name="origin"/>
       <parent link="${parent}_link"/>
-      <child  link="${name}_link"/>
+      <child link="${name}_link"/>
     </joint>
     <!-- gazebo extensions -->

File: pmb2_description/urdf/sensors/structure_sensor.urdf.xacro (robot description, xacro)
@@ -29,7 +29,5 @@
         <origin xyz="0 0 0" rpy="0 0 0"/>
         <!-- inertia tensor computed analytically for a solid cuboid -->
-        <inertia ixx="0.000030"  ixy="0.0"  ixz="0.0"
-                 iyy="0.000030"  iyz="0.0"
-                 izz="0.000002" />
+        <inertia ixx="0.000030" ixy="0.0" ixz="0.0" iyy="0.000030" iyz="0.0" izz="0.000002" />
       </inertial>
       <visual>
@@ -58,7 +56,5 @@
         <mass value="0.01" />
         <origin xyz="0 0 0" rpy="0 0 0"/>
-        <inertia ixx="0.0"  ixy="0.0"  ixz="0.0"
-                 iyy="0.0"  iyz="0.0"
-                 izz="0.0" />
+        <inertia ixx="0.0" ixy="0.0" ixz="0.0" iyy="0.0" iyz="0.0" izz="0.0" />
       </inertial>
     </link>

File: pmb2_description/urdf/wheels/caster.urdf.xacro (robot description, xacro)
@@ -19,7 +19,5 @@
         <origin xyz="-0.00634599 0.00005347 -0.02037519" rpy="0 0 0"/>
         <mass value="0.05144761"/>
-        <inertia  ixx="0.00001513" ixy="-0.00000003" ixz="0.00000267"
-                  iyy="0.00001309" iyz="-0.00000005"
-                  izz="0.00001198"/>
+        <inertia ixx="0.00001513" ixy="-0.00000003" ixz="0.00000267" iyy="0.00001309" iyz="-0.00000005" izz="0.00001198"/>
       </inertial>
       <visual>
@@ -41,8 +39,6 @@
         <origin xyz="0 0 0" rpy="0 0 0"/>
         <mass value="0.08855784"/>
-        <inertia  ixx="0.00001075" ixy="0" ixz="0"
-                  iyy="0.00001541" iyz="0"
-                  izz="0.00001075"/>
-        </inertial>
+        <inertia ixx="0.00001075" ixy="0" ixz="0" iyy="0.00001541" iyz="0" izz="0.00001075"/>
+      </inertial>
       <visual>
         <origin xyz="0 0 0" rpy="0 0 0"/>
@@ -55,5 +51,5 @@
         <origin xyz="0 0 0" rpy="0 0 0"/>
         <geometry>
-	  <sphere radius="${radius}" />
+          <sphere radius="${radius}" />
         </geometry>
       </collision>

File: pmb2_description/urdf/wheels/wheel.urdf.xacro (robot description, xacro)
@@ -19,7 +19,5 @@
         <origin xyz="0 0 ${-0.00207 * reflect}" rpy="0 0 0"/>
         <mass value="1.82362"/>
-        <inertia ixx="0.00499743171" ixy="${ 0.00000004464 * reflect}" ixz="-0.00000002245"
-          iyy="0.00499741733" iyz="${-0.00000000164 * reflect}"
-          izz="0.00839239692"/>
+        <inertia ixx="0.00499743171" ixy="${ 0.00000004464 * reflect}" ixz="-0.00000002245" iyy="0.00499741733" iyz="${-0.00000000164 * reflect}" izz="0.00839239692"/>
       </inertial>
       <visual>
@@ -33,5 +31,6 @@
         <origin xyz="0 0 0" rpy="0 0 0"/>
         <geometry>
-          <sphere radius="${radius}" /> <!-- length="${width}"/> -->
+          <sphere radius="${radius}" />
+          <!-- length="${width}"/> -->
         </geometry>
       </collision>
@@ -41,8 +40,6 @@
         <origin xyz="0 0 -0.02" rpy="0 0 0"/>
         <mass value="10"/>
-        <inertia ixx="1.0" ixy="0" ixz="0"
-                  iyy="1.0" iyz="0"
-                  izz="1.0"/>
-        </inertial>
+        <inertia ixx="1.0" ixy="0" ixz="0" iyy="1.0" iyz="0" izz="1.0"/>
+      </inertial>
       <kinematic>0</kinematic>
       <gravity>1</gravity>
@@ -56,8 +53,5 @@
       <calibration rising="0.0" />
       <dynamics damping="100"/>
-      <safety_controller k_position="0"
-        k_velocity="10"
-        soft_lower_limit="-0.005"
-        soft_upper_limit="0.005" />
+      <safety_controller k_position="0" k_velocity="10" soft_lower_limit="-0.005" soft_upper_limit="0.005" />
     </joint>
     <joint name="wheel_${side}_joint" type="continuous">
