Commit message: Update copyright + move imu into sensors

File: pmb2_description/urdf/base/base.urdf.xacro (robot description, xacro)
@@ -32,5 +32,4 @@
   <xacro:include filename="$(find pmb2_description)/urdf/wheels/wheel.urdf.xacro"/>
   <xacro:include filename="$(find pmb2_description)/urdf/wheels/caster.urdf.xacro"/>
-  <xacro:include filename="$(find pmb2_description)/urdf/sensors/imu.urdf.xacro"/>
   <xacro:include filename="$(find pmb2_description)/urdf/objects/cover.urdf.xacro"/>
   <xacro:include filename="$(find pmb2_description)/urdf/objects/antenna.urdf.xacro"/>

File: pmb2_description/urdf/base/base_sensors.urdf.xacro (robot description, xacro)
@@ -19,4 +19,5 @@
   <!-- INCLUDES -->
   <xacro:include filename="$(find pmb2_description)/urdf/base/base.urdf.xacro"/>
+  <xacro:include filename="$(find pmb2_description)/urdf/sensors/imu.urdf.xacro"/>
   <xacro:include filename="$(find pmb2_description)/urdf/sensors/hokuyo_urg_04lx_ug01_laser.urdf.xacro"/>
   <xacro:include filename="$(find pmb2_description)/urdf/sensors/sick_tim551_laser.urdf.xacro"/>
@@ -26,5 +27,5 @@
   <xacro:include filename="$(find pmb2_description)/urdf/sensors/microphone.urdf.xacro"/>
   <!-- MACRO DEFINITION -->
-  <xacro:macro name="base_sensors" params="name laser_model:=sick-571 sonars:=false has_microphone:=false" >
+  <xacro:macro name="base_sensors" params="name laser_model:=sick-571 has_sonars:=false has_microphone:=false" >
     <!-- IMU -->
     <xacro:imu_sensor name="${name}_imu" parent="${name}_link" update_rate="100.0">

File: pmb2_description/urdf/sensors/bumper.urdf.xacro (robot description, xacro)
@@ -1,5 +1,5 @@
 <?xml version="1.0"?>
 <!--
-  Copyright (c) 2022 PAL Robotics S.L. All rights reserved.
+  Copyright (c) 2024 PAL Robotics S.L. All rights reserved.
   Licensed under the Apache License, Version 2.0 (the "License");
   you may not use this file except in compliance with the License.

File: pmb2_description/urdf/sensors/courier.urdf.xacro (robot description, xacro)
@@ -1,5 +1,5 @@
 <?xml version="1.0"?>
 <!--
-  Copyright (c) 2022 PAL Robotics S.L. All rights reserved.
+  Copyright (c) 2024 PAL Robotics S.L. All rights reserved.
   Licensed under the Apache License, Version 2.0 (the "License");
   you may not use this file except in compliance with the License.

File: pmb2_description/urdf/sensors/elp_rgb.urdf.xacro (robot description, xacro)
@@ -1,5 +1,5 @@
 <?xml version="1.0"?>
 <!--
-  Copyright (c) 2022 PAL Robotics S.L. All rights reserved.
+  Copyright (c) 2024 PAL Robotics S.L. All rights reserved.
   Licensed under the Apache License, Version 2.0 (the "License");
   you may not use this file except in compliance with the License.

File: pmb2_description/urdf/sensors/hokuyo_urg_04lx_ug01_laser.gazebo.xacro (robot description, xacro)
@@ -1,5 +1,5 @@
 <?xml version="1.0"?>
 <!--
-  Copyright (c) 2022 PAL Robotics S.L. All rights reserved.
+  Copyright (c) 2024 PAL Robotics S.L. All rights reserved.
   Licensed under the Apache License, Version 2.0 (the "License");
   you may not use this file except in compliance with the License.

File: pmb2_description/urdf/sensors/hokuyo_urg_04lx_ug01_laser.urdf.xacro (robot description, xacro)
@@ -1,5 +1,5 @@
 <?xml version="1.0"?>
 <!--
-  Copyright (c) 2022 PAL Robotics S.L. All rights reserved.
+  Copyright (c) 2024 PAL Robotics S.L. All rights reserved.
   Licensed under the Apache License, Version 2.0 (the "License");
   you may not use this file except in compliance with the License.

File: pmb2_description/urdf/sensors/microphone.urdf.xacro (robot description, xacro)
@@ -1,5 +1,5 @@
 <?xml version="1.0"?>
 <!--
-  Copyright (c) 2022 PAL Robotics S.L. All rights reserved.
+  Copyright (c) 2024 PAL Robotics S.L. All rights reserved.
   Licensed under the Apache License, Version 2.0 (the "License");
   you may not use this file except in compliance with the License.

File: pmb2_description/urdf/sensors/range.gazebo.xacro (robot description, xacro)
@@ -1,5 +1,5 @@
 <?xml version="1.0"?>
 <!--
-  Copyright (c) 2022 PAL Robotics S.L. All rights reserved.
+  Copyright (c) 2024 PAL Robotics S.L. All rights reserved.
   Licensed under the Apache License, Version 2.0 (the "License");
   you may not use this file except in compliance with the License.

File: pmb2_description/urdf/sensors/range.urdf.xacro (robot description, xacro)
@@ -1,5 +1,5 @@
 <?xml version="1.0"?>
 <!--
-  Copyright (c) 2022 PAL Robotics S.L. All rights reserved.
+  Copyright (c) 2024 PAL Robotics S.L. All rights reserved.
   Licensed under the Apache License, Version 2.0 (the "License");
   you may not use this file except in compliance with the License.

File: pmb2_description/urdf/sensors/sick_tim551_laser.gazebo.xacro (robot description, xacro)
@@ -1,5 +1,5 @@
 <?xml version="1.0"?>
 <!--
-  Copyright (c) 2022 PAL Robotics S.L. All rights reserved.
+  Copyright (c) 2024 PAL Robotics S.L. All rights reserved.
   Licensed under the Apache License, Version 2.0 (the "License");
   you may not use this file except in compliance with the License.

File: pmb2_description/urdf/sensors/sick_tim551_laser.urdf.xacro (robot description, xacro)
@@ -1,5 +1,5 @@
 <?xml version="1.0"?>
 <!--
-  Copyright (c) 2022 PAL Robotics S.L. All rights reserved.
+  Copyright (c) 2024 PAL Robotics S.L. All rights reserved.
   Licensed under the Apache License, Version 2.0 (the "License");
   you may not use this file except in compliance with the License.

File: pmb2_description/urdf/sensors/sick_tim561_laser.gazebo.xacro (robot description, xacro)
@@ -1,5 +1,5 @@
 <?xml version="1.0"?>
 <!--
-  Copyright (c) 2022 PAL Robotics S.L. All rights reserved.
+  Copyright (c) 2024 PAL Robotics S.L. All rights reserved.
   Licensed under the Apache License, Version 2.0 (the "License");
   you may not use this file except in compliance with the License.

File: pmb2_description/urdf/sensors/sick_tim561_laser.urdf.xacro (robot description, xacro)
@@ -1,5 +1,5 @@
 <?xml version="1.0"?>
 <!--
-  Copyright (c) 2022 PAL Robotics S.L. All rights reserved.
+  Copyright (c) 2024 PAL Robotics S.L. All rights reserved.
   Licensed under the Apache License, Version 2.0 (the "License");
   you may not use this file except in compliance with the License.

File: pmb2_description/urdf/sensors/sick_tim571_laser.gazebo.xacro (robot description, xacro)
@@ -1,5 +1,5 @@
 <?xml version="1.0"?>
 <!--
-  Copyright (c) 2022 PAL Robotics S.L. All rights reserved.
+  Copyright (c) 2024 PAL Robotics S.L. All rights reserved.
   Licensed under the Apache License, Version 2.0 (the "License");
   you may not use this file except in compliance with the License.

File: pmb2_description/urdf/sensors/sick_tim571_laser.urdf.xacro (robot description, xacro)
@@ -1,5 +1,5 @@
 <?xml version="1.0"?>
 <!--
-  Copyright (c) 2022 PAL Robotics S.L. All rights reserved.
+  Copyright (c) 2024 PAL Robotics S.L. All rights reserved.
   Licensed under the Apache License, Version 2.0 (the "License");
   you may not use this file except in compliance with the License.

File: pmb2_description/urdf/sensors/structure_sensor.urdf.xacro (robot description, xacro)
@@ -1,5 +1,5 @@
 <?xml version="1.0"?>
 <!--
-  Copyright (c) 2022 PAL Robotics S.L. All rights reserved.
+  Copyright (c) 2024 PAL Robotics S.L. All rights reserved.
   Licensed under the Apache License, Version 2.0 (the "License");
   you may not use this file except in compliance with the License.

File: pmb2_description/urdf/wheels/caster.gazebo.xacro (robot description, xacro)
@@ -1,5 +1,5 @@
 <?xml version="1.0"?>
 <!--
-  Copyright (c) 2022 PAL Robotics S.L. All rights reserved.
+  Copyright (c) 2024 PAL Robotics S.L. All rights reserved.
   Licensed under the Apache License, Version 2.0 (the "License");
   you may not use this file except in compliance with the License.

File: pmb2_description/urdf/wheels/caster.urdf.xacro (robot description, xacro)
@@ -1,5 +1,5 @@
 <?xml version="1.0"?>
 <!--
-  Copyright (c) 2022 PAL Robotics S.L. All rights reserved.
+  Copyright (c) 2024 PAL Robotics S.L. All rights reserved.
   Licensed under the Apache License, Version 2.0 (the "License");
   you may not use this file except in compliance with the License.

File: pmb2_description/urdf/wheels/wheel.urdf.xacro (robot description, xacro)
@@ -1,5 +1,5 @@
 <?xml version="1.0"?>
 <!--
-  Copyright (c) 2022 PAL Robotics S.L. All rights reserved.
+  Copyright (c) 2024 PAL Robotics S.L. All rights reserved.
   Licensed under the Apache License, Version 2.0 (the "License");
   you may not use this file except in compliance with the License.
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
Commit message: Move _link to top file xacro

File: pmb2_description/urdf/base/base.urdf.xacro (robot description, xacro)
@@ -75,11 +75,11 @@
     </xacro:antenna>
     <!-- Wheels -->
-    <xacro:wheel side="right" reflect=" 1.0" radius="${wheel_radius}" width="${wheel_width}" torque="${wheel_torque}" velocity="${wheel_velocity}" separation="${wheel_separation}" parent="${name}"/>
-    <xacro:wheel side="left" reflect="-1.0" radius="${wheel_radius}" width="${wheel_width}" torque="${wheel_torque}" velocity="${wheel_velocity}" separation="${wheel_separation}" parent="${name}"/>
+    <xacro:wheel side="right" reflect=" 1.0" radius="${wheel_radius}" width="${wheel_width}" torque="${wheel_torque}" velocity="${wheel_velocity}" separation="${wheel_separation}" parent="${name}_link"/>
+    <xacro:wheel side="left" reflect="-1.0" radius="${wheel_radius}" width="${wheel_width}" torque="${wheel_torque}" velocity="${wheel_velocity}" separation="${wheel_separation}" parent="${name}_link"/>
     <!-- Casters wheels -->
-    <xacro:caster side="front_right" radius="${caster_radius}" width="${caster_width}" separation_x="${ caster_separation_x}" separation_y="${ caster_separation_y}" offset_x="${caster_offset_x}" offset_y="${caster_offset_y}" offset_z="${caster_offset_z}" parent="${name}"/>
-    <xacro:caster side="front_left" radius="${caster_radius}" width="${caster_width}" separation_x="${ caster_separation_x}" separation_y="${-caster_separation_y}" offset_x="${caster_offset_x}" offset_y="${caster_offset_y}" offset_z="${caster_offset_z}" parent="${name}"/>
-    <xacro:caster side="back_right" radius="${caster_radius}" width="${caster_width}" separation_x="${-caster_separation_x}" separation_y="${ caster_separation_y}" offset_x="${caster_offset_x}" offset_y="${caster_offset_y}" offset_z="${caster_offset_z}" parent="${name}"/>
-    <xacro:caster side="back_left" radius="${caster_radius}" width="${caster_width}" separation_x="${-caster_separation_x}" separation_y="${-caster_separation_y}" offset_x="${caster_offset_x}" offset_y="${caster_offset_y}" offset_z="${caster_offset_z}" parent="${name}"/>
+    <xacro:caster side="front_right" radius="${caster_radius}" width="${caster_width}" separation_x="${ caster_separation_x}" separation_y="${ caster_separation_y}" offset_x="${caster_offset_x}" offset_y="${caster_offset_y}" offset_z="${caster_offset_z}" parent="${name}_link"/>
+    <xacro:caster side="front_left" radius="${caster_radius}" width="${caster_width}" separation_x="${ caster_separation_x}" separation_y="${-caster_separation_y}" offset_x="${caster_offset_x}" offset_y="${caster_offset_y}" offset_z="${caster_offset_z}" parent="${name}_link"/>
+    <xacro:caster side="back_right" radius="${caster_radius}" width="${caster_width}" separation_x="${-caster_separation_x}" separation_y="${ caster_separation_y}" offset_x="${caster_offset_x}" offset_y="${caster_offset_y}" offset_z="${caster_offset_z}" parent="${name}_link"/>
+    <xacro:caster side="back_left" radius="${caster_radius}" width="${caster_width}" separation_x="${-caster_separation_x}" separation_y="${-caster_separation_y}" offset_x="${caster_offset_x}" offset_y="${caster_offset_y}" offset_z="${caster_offset_z}" parent="${name}_link"/>
     <!-- Gazebo config-->
     <xacro:base_gazebo name="${name}"/>

File: pmb2_description/urdf/base/base_sensors.urdf.xacro (robot description, xacro)
@@ -36,5 +36,5 @@
     <xacro:if value="${laser_model == 'hokuyo'}">
       <!-- Theoretic FOV = 220 -->
-      <xacro:hokuyo_urg_04lx_ug01_laser name="${name}_laser" parent="${name}" ros_topic="scan_raw" update_rate="10" min_angle="${-110 * deg_to_rad}" max_angle="${110 * deg_to_rad}">
+      <xacro:hokuyo_urg_04lx_ug01_laser name="${name}_laser" parent="${name}_link" ros_topic="scan_raw" update_rate="10" min_angle="${-110 * deg_to_rad}" max_angle="${110 * deg_to_rad}">
         <origin xyz="${base_laser_x} ${base_laser_y} ${base_laser_z}" rpy="0 0 0" />
       </xacro:hokuyo_urg_04lx_ug01_laser>
@@ -43,5 +43,5 @@
     <xacro:if value="${laser_model == 'sick-551'}">
       <!-- Theoretic FOV = 220 -->
-      <xacro:sick_tim551_laser name="${name}_laser" parent="${name}" ros_topic="scan_raw" update_rate="10" min_angle="${-110 * deg_to_rad}" max_angle="${110 * deg_to_rad}">
+      <xacro:sick_tim551_laser name="${name}_laser" parent="${name}_link" ros_topic="scan_raw" update_rate="10" min_angle="${-110 * deg_to_rad}" max_angle="${110 * deg_to_rad}">
         <origin xyz="${base_laser_x} ${base_laser_y} ${base_laser_z}" rpy="0 0 0" />
       </xacro:sick_tim551_laser>
@@ -50,5 +50,5 @@
     <xacro:if value="${laser_model == 'sick-561'}">
       <!-- Theoretic FOV = 220 -->
-      <xacro:sick_tim561_laser name="${name}_laser" parent="${name}" ros_topic="scan_raw" update_rate="10" min_angle="${-110 * deg_to_rad}" max_angle="${110 * deg_to_rad}">
+      <xacro:sick_tim561_laser name="${name}_laser" parent="${name}_link" ros_topic="scan_raw" update_rate="10" min_angle="${-110 * deg_to_rad}" max_angle="${110 * deg_to_rad}">
         <origin xyz="${base_laser_x} ${base_laser_y} ${base_laser_z}" rpy="0 0 0" />
       </xacro:sick_tim561_laser>
@@ -57,5 +57,5 @@
     <xacro:if value="${laser_model == 'sick-571'}">
       <!-- Theoretic FOV = 220 -->
-      <xacro:sick_tim571_laser name="${name}_laser" parent="${name}" ros_topic="scan_raw" update_rate="10" min_angle="${-110 * deg_to_rad}" max_angle="${110 * deg_to_rad}">
+      <xacro:sick_tim571_laser name="${name}_laser" parent="${name}_link" ros_topic="scan_raw" update_rate="10" min_angle="${-110 * deg_to_rad}" max_angle="${110 * deg_to_rad}">
         <origin xyz="${base_laser_x} ${base_laser_y} ${base_laser_z}" rpy="0 0 0" />
       </xacro:sick_tim571_laser>
@@ -63,11 +63,11 @@
     <!-- Sonars -->
     <xacro:if value="${has_sonars}">
-      <xacro:range_sensor name="${name}_sonar_03" parent="${name}" ros_topic="sonar_${name}" update_rate="5" maxRange="1.0" minRange="0.02" fov="0.5" radiation="ultrasound">
+      <xacro:range_sensor name="${name}_sonar_03" parent="${name}_link" ros_topic="sonar_${name}" update_rate="5" maxRange="1.0" minRange="0.02" fov="0.5" radiation="ultrasound">
         <origin xyz="-0.183 0.183 0.173" rpy="0 0 ${135 * deg_to_rad}"/>
       </xacro:range_sensor>
-      <xacro:range_sensor name="${name}_sonar_02" parent="${name}" ros_topic="sonar_${name}" update_rate="5" maxRange="1.0" minRange="0.02" fov="0.5" radiation="ultrasound">
+      <xacro:range_sensor name="${name}_sonar_02" parent="${name}_link" ros_topic="sonar_${name}" update_rate="5" maxRange="1.0" minRange="0.02" fov="0.5" radiation="ultrasound">
         <origin xyz="-0.259 0.0 0.173" rpy="0 0 ${180 * deg_to_rad}"/>
       </xacro:range_sensor>
-      <xacro:range_sensor name="${name}_sonar_01" parent="${name}" ros_topic="sonar_${name}" update_rate="5" maxRange="1.0" minRange="0.02" fov="0.5" radiation="ultrasound">
+      <xacro:range_sensor name="${name}_sonar_01" parent="${name}_link" ros_topic="sonar_${name}" update_rate="5" maxRange="1.0" minRange="0.02" fov="0.5" radiation="ultrasound">
         <origin xyz="-0.183 -0.183 0.173" rpy="0 0 ${225 * deg_to_rad}"/>
       </xacro:range_sensor>
@@ -75,14 +75,14 @@
     <!-- Microphones -->
     <xacro:if value="${has_microphone}">
-      <xacro:microphone name="${name}_mic_front_left" parent="${name}">
+      <xacro:microphone name="${name}_mic_front_left" parent="${name}_link">
         <origin xyz="0.23182 0.03902 0.195" rpy="0 0 0"/>
       </xacro:microphone>
-      <xacro:microphone name="${name}_mic_front_right" parent="${name}">
+      <xacro:microphone name="${name}_mic_front_right" parent="${name}_link">
         <origin xyz="0.23182 -0.03902 0.195" rpy="0 0 0"/>
       </xacro:microphone>
-      <xacro:microphone name="${name}_mic_back_left" parent="${name}">
+      <xacro:microphone name="${name}_mic_back_left" parent="${name}_link">
         <origin xyz="-0.1082 -0.0599 0.195" rpy="0 0 0"/>
       </xacro:microphone>
-      <xacro:microphone name="${name}_mic_back_right" parent="${name}">
+      <xacro:microphone name="${name}_mic_back_right" parent="${name}_link">
         <origin xyz="-0.1082 -0.13789 0.195" rpy="0 0 0"/>
       </xacro:microphone>

File: pmb2_description/urdf/sensors/bumper.urdf.xacro (robot description, xacro)
@@ -39,5 +39,5 @@
       <axis xyz="0 1 0"/>
       <xacro:insert_block name="origin"/>
-      <parent link="${parent}_link"/>
+      <parent link="${parent}"/>
       <child link="${name}_link"/>
     </joint>

File: pmb2_description/urdf/sensors/courier.urdf.xacro (robot description, xacro)
@@ -38,5 +38,5 @@
   <xacro:property name="rgb_Y" value="0.0   "/>
   <!-- RGBD base -->
-  <xacro:structure_sensor name="base_rgbd_camera" parent="base">
+  <xacro:structure_sensor name="base_rgbd_camera" parent="base_link">
     <!-- Pose of sensor frame wrt to base -->
     <origin xyz="${base_rgbd_x} ${base_rgbd_y} ${base_rgbd_z}" rpy="${base_rgbd_R * deg_to_rad} ${base_rgbd_P * deg_to_rad} ${base_rgbd_Y * deg_to_rad}"/>
@@ -45,5 +45,5 @@
   </xacro:structure_sensor>
   <!-- RGBD roof -->
-  <xacro:structure_sensor name="roof_rgbd_camera" parent="base">
+  <xacro:structure_sensor name="roof_rgbd_camera" parent="base_link">
     <!-- Pose of sensor frame wrt to base -->
     <origin xyz="${roof_rgbd_x} ${roof_rgbd_y} ${roof_rgbd_z}" rpy="${roof_rgbd_R * deg_to_rad} ${roof_rgbd_P * deg_to_rad} ${roof_rgbd_Y * deg_to_rad}"/>
@@ -52,5 +52,5 @@
   </xacro:structure_sensor>
   <!-- RGB -->
-  <xacro:elp_rgb name="rgb_camera" parent="base">
+  <xacro:elp_rgb name="rgb_camera" parent="base_link">
     <!-- Pose of sensor frame wrt to base -->
     <origin xyz="${rgb_x} ${rgb_y} ${rgb_z}" rpy="${rgb_R * deg_to_rad} ${rgb_P * deg_to_rad} ${rgb_Y * deg_to_rad}"/>

File: pmb2_description/urdf/sensors/elp_rgb.urdf.xacro (robot description, xacro)
@@ -20,5 +20,5 @@
       <xacro:insert_block name="origin"/>
       <axis xyz="0 0 1"/>
-      <parent link="${parent}_link"/>
+      <parent link="${parent}"/>
       <child link="${name}_link"/>
     </joint>

File: pmb2_description/urdf/sensors/hokuyo_urg_04lx_ug01_laser.urdf.xacro (robot description, xacro)
@@ -32,5 +32,5 @@
       <axis xyz="0 1 0"/>
       <xacro:insert_block name="origin"/>
-      <parent link="${parent}_link"/>
+      <parent link="${parent}"/>
       <child link="${name}_link"/>
     </joint>

File: pmb2_description/urdf/sensors/microphone.urdf.xacro (robot description, xacro)
@@ -19,5 +19,5 @@
       <xacro:insert_block name="origin"/>
       <child link="${name}_link"/>
-      <parent link="${parent}_link"/>
+      <parent link="${parent}"/>
     </joint>
   </xacro:macro>

File: pmb2_description/urdf/sensors/range.urdf.xacro (robot description, xacro)
@@ -32,5 +32,5 @@
       <xacro:insert_block name="origin"/>
       <axis xyz="0 0 1"/>
-      <parent link="${parent}_link"/>
+      <parent link="${parent}"/>
       <child link="${name}_link"/>
     </joint>

File: pmb2_description/urdf/sensors/sick_tim551_laser.urdf.xacro (robot description, xacro)
@@ -32,5 +32,5 @@
       <axis xyz="0 1 0"/>
       <xacro:insert_block name="origin"/>
-      <parent link="${parent}_link"/>
+      <parent link="${parent}"/>
       <child link="${name}_link"/>
     </joint>

File: pmb2_description/urdf/sensors/sick_tim561_laser.urdf.xacro (robot description, xacro)
@@ -32,5 +32,5 @@
       <axis xyz="0 1 0"/>
       <xacro:insert_block name="origin"/>
-      <parent link="${parent}_link"/>
+      <parent link="${parent}"/>
       <child link="${name}_link"/>
     </joint>

File: pmb2_description/urdf/sensors/sick_tim571_laser.urdf.xacro (robot description, xacro)
@@ -32,5 +32,5 @@
       <axis xyz="0 1 0"/>
       <xacro:insert_block name="origin"/>
-      <parent link="${parent}_link"/>
+      <parent link="${parent}"/>
       <child link="${name}_link"/>
     </joint>

File: pmb2_description/urdf/sensors/structure_sensor.urdf.xacro (robot description, xacro)
@@ -21,5 +21,5 @@
       <axis xyz="0 0 1"/>
       <!-- <limit lower="0" upper="0.001" effort="100" velocity="0.01"/> -->
-      <parent link="${parent}_link"/>
+      <parent link="${parent}"/>
       <child link="${name}_link"/>
     </joint>

File: pmb2_description/urdf/wheels/caster.urdf.xacro (robot description, xacro)
@@ -56,5 +56,5 @@
     </link>
     <joint name="caster_${side}_1_joint" type="continuous">
-      <parent link="${parent}_link"/>
+      <parent link="${parent}"/>
       <child link="caster_${side}_1_link"/>
       <origin xyz="${offset_x + separation_x / 2} ${offset_y - separation_y / 2} ${offset_z}" rpy="0 0 0"/>

File: pmb2_description/urdf/wheels/wheel.urdf.xacro (robot description, xacro)
@@ -50,5 +50,5 @@
       <limit effort="100.0" lower="-0.005" upper="0.005" velocity="1.0"/>
       <child link="suspension_${side}_link"/>
-      <parent link="${parent}_link"/>
+      <parent link="${parent}"/>
       <calibration rising="0.0" />
       <dynamics damping="100"/>
