Commit message: Set casters and suspension joints to fixed

File: pmb2_description/urdf/wheels/caster.gazebo.xacro (robot description, xacro)
@@ -18,10 +18,6 @@
       <kp>1000000.0</kp>
       <kd>10000.0</kd>
-      <friction>
-        <ode>
-          <mu>1.0</mu>
-          <mu2>1.0</mu2>
-        </ode>
-      </friction>
+      <mu1>0.0</mu1>
+      <mu2>0.0</mu2>
       <!--<fdir1>1 0 0</fdir1>-->
       <max_vel>1.0</max_vel>
@@ -32,10 +28,6 @@
       <kp>1000000.0</kp>
       <kd>10000.0</kd>
-      <friction>
-        <ode>
-          <mu>1.0</mu>
-          <mu2>1.0</mu2>
-        </ode>
-      </friction>
+      <mu1>0.0</mu1>
+      <mu2>0.0</mu2>
       <!--<fdir1>1 0 0</fdir1>-->
       <max_vel>1.0</max_vel>

File: pmb2_description/urdf/wheels/caster.urdf.xacro (robot description, xacro)
@@ -55,17 +55,15 @@
       </collision>
     </link>
-    <joint name="caster_${side}_1_joint" type="continuous">
+    <joint name="caster_${side}_1_joint" type="fixed">
       <parent link="${parent}"/>
       <child link="caster_${side}_1_link"/>
       <origin xyz="${offset_x + separation_x / 2} ${offset_y - separation_y / 2} ${offset_z}" rpy="0 0 0"/>
       <axis xyz="0 0 1"/>
-      <dynamics damping="0.015" friction="0.0"/>
     </joint>
-    <joint name="caster_${side}_2_joint" type="continuous">
+    <joint name="caster_${side}_2_joint" type="fixed">
       <parent link="caster_${side}_1_link"/>
       <child link="caster_${side}_2_link"/>
       <origin xyz="-0.016 0.0000 -0.040" rpy="${-90.0 * deg_to_rad} 0 0"/>
       <axis xyz="0 0 1"/>
-      <dynamics damping="0.015" friction="0.0"/>
     </joint>
     <!-- Gazebo extensions -->

File: pmb2_description/urdf/wheels/wheel.urdf.xacro (robot description, xacro)
@@ -45,13 +45,9 @@
       <gravity>1</gravity>
     </link>
-    <joint name="suspension_${side}_joint" type="prismatic">
+    <joint name="suspension_${side}_joint" type="fixed">
       <origin xyz="0 0 0" rpy="0 0 0"/>
       <axis xyz="0 0 1"/>
-      <limit effort="100.0" lower="-0.005" upper="0.005" velocity="1.0"/>
       <child link="suspension_${side}_link"/>
       <parent link="${parent}"/>
-      <calibration rising="0.0" />
-      <dynamics damping="100"/>
-      <safety_controller k_position="0" k_velocity="10" soft_lower_limit="-0.005" soft_upper_limit="0.005" />
     </joint>
     <joint name="wheel_${side}_joint" type="continuous">
