Commit message: Cleaning and proper main structure

File: pmb2_description/robots/pmb2.urdf.xacro (robot description, xacro)
@@ -1,5 +1,5 @@
 <?xml version="1.0"?>
 <!--
-  Copyright (c) 2022 PAL Robotics S.L. All rights reserved.
+  Copyright (c) 2024 PAL Robotics S.L. All rights reserved.
   Licensed under the Apache License, Version 2.0 (the "License");
   you may not use this file except in compliance with the License.
@@ -11,36 +11,54 @@
   See the License for the specific language governing permissions and
   limitations under the License.
- -->
-<robot  xmlns:xacro="http://ros.org/wiki/xacro"
-        name="pmb2" >
-  <xacro:arg name="use_sim" default="false"/>
-  <xacro:arg name="laser_model" default="sick-571"/> <!-- no-laser, hokuyo, sick-551, sick-561, sick-571-->
-  <xacro:arg name="courier_rgbd_sensors" default="false"/> <!-- false, true-->
+-->
+<robot xmlns:xacro="http://ros.org/wiki/xacro" name="pmb2">
+  <!-- ARGUMENTS -->
+  <!-- no-laser, hokuyo, sick-551, sick-561, sick-571-->
+  <xacro:arg name="laser_model" default="sick-571"/>
+  <!-- false, true -->
+  <xacro:arg name="has_sonars" default="true"/>
+  <!-- false, true -->
+  <xacro:arg name="has_microphone" default="false"/>
+  <!-- false, true-->
+  <xacro:arg name="has_courier_rgbd_sensors" default="false"/>
+  <!-- Execution env config -->
+  <xacro:arg name="use_sim_time" default="false"/>
+  <xacro:arg name="is_multiple" default="false"/>
+  <xacro:arg name=" namespace" default=""/>
+  <xacro:arg name="is_public_sim" default="false"/>
+  <!-- PROPERTIES -->
+  <!-- HW configuration -->
   <xacro:property name="laser_model" value="$(arg laser_model)" />
-  <xacro:property name="courier_rgbd_sensors" value="$(arg courier_rgbd_sensors)"/>
+  <xacro:property name="has_sonars" value="$(arg has_sonars)" />
+  <xacro:property name="has_microphone" value="$(arg has_microphone)" />
+  <xacro:property name="has_courier_rgbd_sensors" value="$(arg has_courier_rgbd_sensors)"/>
+  <!-- HW configuration check -->
   <xacro:if value="${laser_model not in ['no-laser', 'sick-551', 'sick-561', 'sick-571', 'hokuyo']}">
     <xacro:wrong_laser_model/>
   </xacro:if>
-  <xacro:arg name="multiple" default="false"/>
-  <xacro:arg name="namespace" default=""/>
-  <xacro:property name="is_multiple" value="$(arg multiple)" />
-  <xacro:property name="nsp" value="$(arg namespace)" />
-  <!-- The following included files set up definitions of parts of the robot body -->
+  <!-- Execution env configuration -->
+  <xacro:property name="use_sim_time" default="$(arg use_sim_time)"/>
+  <xacro:property name="is_multiple" value="$(arg is_multiple)" />
+  <xacro:property name="namespace" value="$(arg namespace)" />
+  <xacro:property name="is_public_sim" value="$(arg is_public_sim)" />
+  <!-- INCLUDES -->
   <!-- Base -->
   <xacro:include filename="$(find pmb2_description)/urdf/base/base_sensors.urdf.xacro" />
-  <!-- Generic simulator_gazebo plugins -->
-  <xacro:include filename="$(find pmb2_description)/gazebo/gazebo.urdf.xacro" />
-  <!-- ros2_control -->
-  <xacro:include filename="$(find pmb2_description)/ros2_control/ros2_control.urdf.xacro" />
-  <xacro:pmb2_ros2_control
-    use_sim="$(arg use_sim)" />
+  <!-- Courier rgbd sensors -->
+  <xacro:if value="${has_courier_rgbd_sensors}">
+    <xacro:include filename="$(find pmb2_description)/urdf/cameras_add_on/cameras_add_on.urdf.xacro" />
+  </xacro:if>
   <!-- Materials for visualization -->
   <xacro:include filename="$(find pal_urdf_utils)/urdf/materials.urdf.xacro" />
+  <!-- ROS 2 Control -->
+  <xacro:include filename="$(find pmb2_description)/ros2_control/ros2_control.urdf.xacro" />
+  <!-- ROBOT DEFINITION -->
   <!-- Now we can start using the macros included above to define the actual robot -->
-  <xacro:base_sensors name="base" laser_model="$(arg laser_model)" sonars="true"/>
+  <xacro:base_sensors name="base"/>
   <!-- RGBD Sensors -->
-  <xacro:if value="${courier_rgbd_sensors}">
-    <xacro:include filename="$(find pmb2_description)/urdf/cameras_add_on/cameras_add_on.urdf.xacro" />
+  <xacro:if value="${has_courier_rgbd_sensors}">
     <xacro:cameras_add_on name="cameras_add_on" parent="base_link"/>
   </xacro:if>
+  <!-- ROS 2 Control -->
+  <xacro:pmb2_ros2_control />
 </robot>

File: pmb2_description/ros2_control/ros2_control.urdf.xacro (robot description, xacro)
@@ -1,5 +1,5 @@
 <?xml version="1.0"?>
 <!--
-Copyright (c) 2022 PAL Robotics S.L. All rights reserved.
+Copyright (c) 2024 PAL Robotics S.L. All rights reserved.
 Licensed under the Apache License, Version 2.0 (the "License");
 you may not use this file except in compliance with the License.
@@ -12,17 +12,31 @@
 limitations under the License.
  -->
-<robot xmlns:xacro="http://ros.org/wiki/xacro"
-       name="pmb2" >
-<xacro:macro name="pmb2_ros2_control" params="use_sim:=^|false">
-    <xacro:include filename="$(find pmb2_description)/urdf/wheels/wheel.ros2_control.xacro"/>
-    <xacro:include filename="$(find pmb2_description)/urdf/sensors/sensors.ros2_control.xacro"/>
+<robot xmlns:xacro="http://ros.org/wiki/xacro" name="pmb2">
+  <!-- INCLUDES -->
+  <xacro:include filename="$(find pmb2_description)/urdf/wheels/wheel.ros2_control.xacro"/>
+  <xacro:include filename="$(find pmb2_description)/urdf/sensors/sensors.ros2_control.xacro"/>
+  <!-- MACRO DEFINITION-->
+  <xacro:macro name="pmb2_ros2_control">
+    <!-- Init the ROS 2 control gazebo interface -->
+    <xacro:if value="${use_sim_time}">
+      <gazebo>
+        <plugin filename="libgazebo_ros2_control.so" name="gazebo_ros2_control">
+          <parameters>$(find pmb2_description)/ros2_control/gazebo_controller_manager_cfg.yaml</parameters>
+        </plugin>
+      </gazebo>
+    </xacro:if>
+    <!-- ROS 2 control config-->
     <ros2_control name="ros2_control_pmb2_system" type="system">
-      <xacro:if value="$(arg use_sim)">
-        <xacro:ros2_control_imu name="base_imu_sensor"/>
+      <!-- Execution env config -->
+      <xacro:if value="${use_sim_time}">
+        <!-- HW interface: gazebo-->
         <hardware>
           <plugin>gazebo_ros2_control/GazeboSystem</plugin>
         </hardware>
+        <!-- IMU sensor (only in simulation)-->
+        <xacro:ros2_control_imu name="base_imu_sensor"/>
       </xacro:if>
-      <xacro:unless value="$(arg use_sim)">
+      <xacro:unless value="${use_sim_time}">
+        <!-- HW interface: robot control-->
         <hardware>
           <plugin>robot_control/RobotControl</plugin>

File: pmb2_description/urdf/base/base.urdf.xacro (robot description, xacro)
@@ -1,5 +1,5 @@
 <?xml version="1.0"?>
 <!--
-  Copyright (c) 2022 PAL Robotics S.L. All rights reserved.
+  Copyright (c) 2024 PAL Robotics S.L. All rights reserved.
   Licensed under the Apache License, Version 2.0 (the "License");
   you may not use this file except in compliance with the License.
@@ -11,12 +11,7 @@
   See the License for the specific language governing permissions and
   limitations under the License.
- -->
+-->
 <robot xmlns:xacro="http://ros.org/wiki/xacro">
-  <xacro:include filename="$(find pal_urdf_utils)/urdf/deg_to_rad.urdf.xacro"/>
-  <xacro:include filename="$(find pmb2_description)/urdf/wheels/wheel.urdf.xacro"/>
-  <xacro:include filename="$(find pmb2_description)/urdf/wheels/caster.urdf.xacro"/>
-  <xacro:include filename="$(find pmb2_description)/urdf/sensors/imu.urdf.xacro"/>
-  <xacro:include filename="$(find pmb2_description)/urdf/objects/cover.urdf.xacro"/>
-  <xacro:include filename="$(find pmb2_description)/urdf/objects/antenna.urdf.xacro"/>
+  <!-- PROPERTIES -->
   <!-- Wheel characteristics -->
   <xacro:property name="wheel_radius" value="0.0985"/>
@@ -33,4 +28,13 @@
   <xacro:property name="caster_offset_y" value="0.0"/>
   <xacro:property name="caster_offset_z" value="-0.0335"/>
+  <!-- INCLUDES -->
+  <xacro:include filename="$(find pal_urdf_utils)/urdf/deg_to_rad.urdf.xacro"/>
+  <xacro:include filename="$(find pmb2_description)/urdf/base/base.gazebo.xacro"/>
+  <xacro:include filename="$(find pmb2_description)/urdf/wheels/wheel.urdf.xacro"/>
+  <xacro:include filename="$(find pmb2_description)/urdf/wheels/caster.urdf.xacro"/>
+  <xacro:include filename="$(find pmb2_description)/urdf/sensors/imu.urdf.xacro"/>
+  <xacro:include filename="$(find pmb2_description)/urdf/objects/cover.urdf.xacro"/>
+  <xacro:include filename="$(find pmb2_description)/urdf/objects/antenna.urdf.xacro"/>
+  <!-- MACRO DEFINITION-->
   <xacro:macro name="base" params="name">
     <!-- Base -->
@@ -56,7 +60,4 @@
       </collision>
     </link>
-    <gazebo reference="${name}_link">
-      <material>Gazebo/White</material>
-    </gazebo>
     <!-- Base footprint -->
     <link name="${name}_footprint"/>
@@ -66,17 +67,7 @@
       <parent link="${name}_footprint"/>
     </joint>
-    <!-- gazebo parameters are given here for base_link thru base_footprint -->
-    <gazebo reference="${name}_footprint">
-      <kp>100000000.0</kp>
-      <kd>10.0</kd>
-      <mu1>0.1</mu1>
-      <mu2>0.1</mu2>
-      <fdir1>1 0 0</fdir1>
-      <maxVel>10.0</maxVel>
-      <minDepth>0.0005</minDepth>
-      <laserRetro>0</laserRetro>
-    </gazebo>
-    <!-- Orange cover & antennas -->
+    <!-- Orange cover -->
     <xacro:cover name="${name}_cover" parent="${name}_footprint"/>
+    <!-- Antennas -->
     <xacro:antenna name="${name}_antenna_left" parent="${name}_link">
       <origin xyz="-0.201 0.1062 0.195" rpy="0 0 0"/>
@@ -85,8 +76,4 @@
       <origin xyz="-0.201 -0.1062 0.195" rpy="0 0 0"/>
     </xacro:antenna>
-    <!-- IMU -->
-    <xacro:imu_sensor name="${name}_imu" parent="${name}_link" update_rate="100.0">
-      <origin xyz="0.10171 0 0.11282" rpy="0 0 ${-90 * deg_to_rad}"/>
-    </xacro:imu_sensor>
     <!-- Wheels -->
     <xacro:wheel side="right" reflect=" 1.0" radius="${wheel_radius}" width="${wheel_width}" torque="${wheel_torque}" velocity="${wheel_velocity}" separation="${wheel_separation}" parent="${name}"/>
@@ -97,4 +84,6 @@
     <xacro:caster side="back_right" radius="${caster_radius}" width="${caster_width}" separation_x="${-caster_separation_x}" separation_y="${ caster_separation_y}" offset_x="${caster_offset_x}" offset_y="${caster_offset_y}" offset_z="${caster_offset_z}" parent="${name}"/>
     <xacro:caster side="back_left" radius="${caster_radius}" width="${caster_width}" separation_x="${-caster_separation_x}" separation_y="${-caster_separation_y}" offset_x="${caster_offset_x}" offset_y="${caster_offset_y}" offset_z="${caster_offset_z}" parent="${name}"/>
+    <!-- Gazebo config-->
+    <xacro:base_gazebo name="${name}"/>
   </xacro:macro>
 </robot>

File: pmb2_description/urdf/base/base_sensors.urdf.xacro (robot description, xacro)
@@ -11,5 +11,5 @@
   See the License for the specific language governing permissions and
   limitations under the License.
- -->
+-->
 <robot xmlns:xacro="http://ros.org/wiki/xacro">
   <!-- PROPERTIES -->
@@ -26,35 +26,42 @@
   <xacro:include filename="$(find pmb2_description)/urdf/sensors/microphone.urdf.xacro"/>
   <!-- MACRO DEFINITION -->
-  <xacro:macro name="base_sensors" params=" name laser_model:=sick-571 sonars:=false microphone:=false ">
-    <xacro:if value="${laser_model == 'hokuyo'}">
-      <!-- Laser -->
-      <!-- Theoretic FOV = 220 -->
-      <xacro:hokuyo_urg_04lx_ug01_laser name="${name}_laser" parent="${name}" ros_topic="scan_raw" update_rate="10" min_angle="${-110 * deg_to_rad}" max_angle="${110 * deg_to_rad}">
-        <origin xyz="${base_laser_x} ${base_laser_y} ${base_laser_z}" rpy="0 0 0" />
-      </xacro:hokuyo_urg_04lx_ug01_laser>
+  <xacro:macro name="base_sensors" params="name">
+    <!-- IMU -->
+    <xacro:imu_sensor name="${name}_imu" parent="${name}_link" update_rate="100.0">
+      <origin xyz="0.10171 0 0.11282" rpy="0 0 ${-90 * deg_to_rad}"/>
+    </xacro:imu_sensor>
+    <!-- Laser -->
+    <xacro:if value="${laser_model != 'no-laser'}">
+      <!-- Hokuyo -->
+      <xacro:if value="${laser_model == 'hokuyo'}">
+        <!-- Theoretic FOV = 220 -->
+        <xacro:hokuyo_urg_04lx_ug01_laser name="${name}_laser" parent="${name}" ros_topic="scan_raw" update_rate="10" min_angle="${-110 * deg_to_rad}" max_angle="${110 * deg_to_rad}">
+          <origin xyz="${base_laser_x} ${base_laser_y} ${base_laser_z}" rpy="0 0 0" />
+        </xacro:hokuyo_urg_04lx_ug01_laser>
+      </xacro:if>
+      <!-- sick-551 -->
+      <xacro:if value="${laser_model == 'sick-551'}">
+        <!-- Theoretic FOV = 220 -->
+        <xacro:sick_tim551_laser name="${name}_laser" parent="${name}" ros_topic="scan_raw" update_rate="10" min_angle="${-110 * deg_to_rad}" max_angle="${110 * deg_to_rad}">
+          <origin xyz="${base_laser_x} ${base_laser_y} ${base_laser_z}" rpy="0 0 0" />
+        </xacro:sick_tim551_laser>
+      </xacro:if>
+      <!-- sick-561 -->
+      <xacro:if value="${laser_model == 'sick-561'}">
+        <!-- Theoretic FOV = 220 -->
+        <xacro:sick_tim561_laser name="${name}_laser" parent="${name}" ros_topic="scan_raw" update_rate="10" min_angle="${-110 * deg_to_rad}" max_angle="${110 * deg_to_rad}">
+          <origin xyz="${base_laser_x} ${base_laser_y} ${base_laser_z}" rpy="0 0 0" />
+        </xacro:sick_tim561_laser>
+      </xacro:if>
+      <!-- sick-571 -->
+      <xacro:if value="${laser_model == 'sick-571'}">
+        <!-- Theoretic FOV = 220 -->
+        <xacro:sick_tim571_laser name="${name}_laser" parent="${name}" ros_topic="scan_raw" update_rate="10" min_angle="${-110 * deg_to_rad}" max_angle="${110 * deg_to_rad}">
+          <origin xyz="${base_laser_x} ${base_laser_y} ${base_laser_z}" rpy="0 0 0" />
+        </xacro:sick_tim571_laser>
+      </xacro:if>
     </xacro:if>
-    <xacro:if value="${laser_model == 'sick-551'}">
-      <!-- Laser -->
-      <!-- Theoretic FOV = 220 -->
-      <xacro:sick_tim551_laser name="${name}_laser" parent="${name}" ros_topic="scan_raw" update_rate="10" min_angle="${-110 * deg_to_rad}" max_angle="${110 * deg_to_rad}">
-        <origin xyz="${base_laser_x} ${base_laser_y} ${base_laser_z}" rpy="0 0 0" />
-      </xacro:sick_tim551_laser>
-    </xacro:if>
-    <xacro:if value="${laser_model == 'sick-561'}">
-      <!-- Laser -->
-      <!-- Theoretic FOV = 220 -->
-      <xacro:sick_tim561_laser name="${name}_laser" parent="${name}" ros_topic="scan_raw" update_rate="10" min_angle="${-110 * deg_to_rad}" max_angle="${110 * deg_to_rad}">
-        <origin xyz="${base_laser_x} ${base_laser_y} ${base_laser_z}" rpy="0 0 0" />
-      </xacro:sick_tim561_laser>
-    </xacro:if>
-    <xacro:if value="${laser_model == 'sick-571'}">
-      <!-- Laser -->
-      <!-- Theoretic FOV = 220 -->
-      <xacro:sick_tim571_laser name="${name}_laser" parent="${name}" ros_topic="scan_raw" update_rate="10" min_angle="${-110 * deg_to_rad}" max_angle="${110 * deg_to_rad}">
-        <origin xyz="${base_laser_x} ${base_laser_y} ${base_laser_z}" rpy="0 0 0" />
-      </xacro:sick_tim571_laser>
-    </xacro:if>
-    <xacro:if value="${sonars}">
-      <!-- Sonars -->
+    <!-- Sonars -->
+    <xacro:if value="${has_sonars}">
       <xacro:range_sensor name="${name}_sonar_03" parent="${name}" ros_topic="sonar_${name}" update_rate="5" maxRange="1.0" minRange="0.02" fov="0.5" radiation="ultrasound">
         <origin xyz="-0.183 0.183 0.173" rpy="0 0 ${135 * deg_to_rad}"/>
@@ -67,6 +74,6 @@
       </xacro:range_sensor>
     </xacro:if>
-    <xacro:if value="${microphone}">
-      <!-- Microphones -->
+    <!-- Microphones -->
+    <xacro:if value="${has_microphone}">
       <xacro:microphone name="${name}_mic_front_left" parent="${name}">
         <origin xyz="0.23182 0.03902 0.195" rpy="0 0 0"/>

File: pmb2_description/urdf/cameras_add_on/cameras_add_on.urdf.xacro (robot description, xacro)
@@ -8,30 +8,28 @@
         <origin xyz="-0.00001132 0.04392363 0.06783541" rpy="0.0 0.0 0.0"/>
         <mass value="3.057"/>
-        <inertia ixx="0.08241443" ixy="-0.00000558" ixz="-0.00001319"
-          iyy="0.05540468" iyz="0.01732357"
-          izz="0.07634613"/>
-        </inertial>
-        <visual>
-          <origin xyz="0 0 0" rpy="0 0 0"/>
-          <geometry>
-            <mesh filename="package://pmb2_description/meshes/cameras_add_on/cameras_add_on.stl" scale="1 1 1"/>
-          </geometry>
-          <material name="White" />
-        </visual>
-        <collision>
-          <origin xyz="0 0 0" rpy="0 0 0" />
-          <geometry>
-            <mesh filename="package://pmb2_description/meshes/cameras_add_on/cameras_add_on_collision.stl" scale="1 1 1"/>
-          </geometry>
-          <material name="White" />
-        </collision>
-      </link>
-      <joint name="${name}_joint" type="fixed">
-        <parent link="${parent}"/>
-        <child link="${name}_link"/>
-        <origin xyz="0.0 0.0 0.0"  rpy="0 0 0" />
-        <axis xyz="0 0 1" />
-      </joint>
-    </xacro:macro>
-    <xacro:include filename="$(find pmb2_description)/urdf/sensors/courier.urdf.xacro" />
-  </robot>
+        <inertia ixx="0.08241443" ixy="-0.00000558" ixz="-0.00001319" iyy="0.05540468" iyz="0.01732357" izz="0.07634613"/>
+      </inertial>
+      <visual>
+        <origin xyz="0 0 0" rpy="0 0 0"/>
+        <geometry>
+          <mesh filename="package://pmb2_description/meshes/cameras_add_on/cameras_add_on.stl" scale="1 1 1"/>
+        </geometry>
+        <material name="White" />
+      </visual>
+      <collision>
+        <origin xyz="0 0 0" rpy="0 0 0" />
+        <geometry>
+          <mesh filename="package://pmb2_description/meshes/cameras_add_on/cameras_add_on_collision.stl" scale="1 1 1"/>
+        </geometry>
+        <material name="White" />
+      </collision>
+    </link>
+    <joint name="${name}_joint" type="fixed">
+      <parent link="${parent}"/>
+      <child link="${name}_link"/>
+      <origin xyz="0.0 0.0 0.0" rpy="0 0 0" />
+      <axis xyz="0 0 1" />
+    </joint>
+  </xacro:macro>
+  <xacro:include filename="$(find pmb2_description)/urdf/sensors/courier.urdf.xacro" />
+</robot>

Commit message: Bring back the parameters

File: pmb2_description/robots/pmb2.urdf.xacro (robot description, xacro)
@@ -55,5 +55,5 @@
   <!-- ROBOT DEFINITION -->
   <!-- Now we can start using the macros included above to define the actual robot -->
-  <xacro:base_sensors name="base"/>
+  <xacro:base_sensors name="base" laser_model="$(arg laser_model)" sonars="true" has_microphone="$(arg has_microphone)"/>
   <!-- RGBD Sensors -->
   <xacro:if value="${has_courier_rgbd_sensors}">

File: pmb2_description/urdf/base/base_sensors.urdf.xacro (robot description, xacro)
@@ -26,5 +26,5 @@
   <xacro:include filename="$(find pmb2_description)/urdf/sensors/microphone.urdf.xacro"/>
   <!-- MACRO DEFINITION -->
-  <xacro:macro name="base_sensors" params="name">
+  <xacro:macro name="base_sensors" params="name laser_model:=sick-571 sonars:=false has_microphone:=false" >
     <!-- IMU -->
     <xacro:imu_sensor name="${name}_imu" parent="${name}_link" update_rate="100.0">
