Commit message: URDF cleanup

File: pmb2_description/robots/pmb2.urdf.xacro (robot description, xacro)
@@ -55,4 +55,5 @@
   <!-- ROS 2 Control -->
   <xacro:include filename="$(find pmb2_description)/ros2_control/ros2_control.urdf.xacro" />
+  <xacro:pmb2_ros2_control />
   <!-- ROBOT DEFINITION -->
   <!-- Now we can start using the macros included above to define the actual robot -->
@@ -62,5 +63,3 @@
     <xacro:cameras_add_on name="cameras_add_on" parent="base_link"/>
   </xacro:if>
-  <!-- ROS 2 Control -->
-  <xacro:pmb2_ros2_control />
 </robot>

File: pmb2_description/urdf/base/base_sensors.urdf.xacro (robot description, xacro)
@@ -33,33 +33,31 @@
     </xacro:imu_sensor>
     <!-- Laser -->
-    <xacro:if value="${laser_model != 'no-laser'}">
-      <!-- Hokuyo -->
-      <xacro:if value="${laser_model == 'hokuyo'}">
-        <!-- Theoretic FOV = 220 -->
-        <xacro:hokuyo_urg_04lx_ug01_laser name="${name}_laser" parent="${name}" ros_topic="scan_raw" update_rate="10" min_angle="${-110 * deg_to_rad}" max_angle="${110 * deg_to_rad}">
-          <origin xyz="${base_laser_x} ${base_laser_y} ${base_laser_z}" rpy="0 0 0" />
-        </xacro:hokuyo_urg_04lx_ug01_laser>
-      </xacro:if>
-      <!-- sick-551 -->
-      <xacro:if value="${laser_model == 'sick-551'}">
-        <!-- Theoretic FOV = 220 -->
-        <xacro:sick_tim551_laser name="${name}_laser" parent="${name}" ros_topic="scan_raw" update_rate="10" min_angle="${-110 * deg_to_rad}" max_angle="${110 * deg_to_rad}">
-          <origin xyz="${base_laser_x} ${base_laser_y} ${base_laser_z}" rpy="0 0 0" />
-        </xacro:sick_tim551_laser>
-      </xacro:if>
-      <!-- sick-561 -->
-      <xacro:if value="${laser_model == 'sick-561'}">
-        <!-- Theoretic FOV = 220 -->
-        <xacro:sick_tim561_laser name="${name}_laser" parent="${name}" ros_topic="scan_raw" update_rate="10" min_angle="${-110 * deg_to_rad}" max_angle="${110 * deg_to_rad}">
-          <origin xyz="${base_laser_x} ${base_laser_y} ${base_laser_z}" rpy="0 0 0" />
-        </xacro:sick_tim561_laser>
-      </xacro:if>
-      <!-- sick-571 -->
-      <xacro:if value="${laser_model == 'sick-571'}">
-        <!-- Theoretic FOV = 220 -->
-        <xacro:sick_tim571_laser name="${name}_laser" parent="${name}" ros_topic="scan_raw" update_rate="10" min_angle="${-110 * deg_to_rad}" max_angle="${110 * deg_to_rad}">
-          <origin xyz="${base_laser_x} ${base_laser_y} ${base_laser_z}" rpy="0 0 0" />
-        </xacro:sick_tim571_laser>
-      </xacro:if>
+    <!-- Hokuyo -->
+    <xacro:if value="${laser_model == 'hokuyo'}">
+      <!-- Theoretic FOV = 220 -->
+      <xacro:hokuyo_urg_04lx_ug01_laser name="${name}_laser" parent="${name}" ros_topic="scan_raw" update_rate="10" min_angle="${-110 * deg_to_rad}" max_angle="${110 * deg_to_rad}">
+        <origin xyz="${base_laser_x} ${base_laser_y} ${base_laser_z}" rpy="0 0 0" />
+      </xacro:hokuyo_urg_04lx_ug01_laser>
+    </xacro:if>
+    <!-- sick-551 -->
+    <xacro:if value="${laser_model == 'sick-551'}">
+      <!-- Theoretic FOV = 220 -->
+      <xacro:sick_tim551_laser name="${name}_laser" parent="${name}" ros_topic="scan_raw" update_rate="10" min_angle="${-110 * deg_to_rad}" max_angle="${110 * deg_to_rad}">
+        <origin xyz="${base_laser_x} ${base_laser_y} ${base_laser_z}" rpy="0 0 0" />
+      </xacro:sick_tim551_laser>
+    </xacro:if>
+    <!-- sick-561 -->
+    <xacro:if value="${laser_model == 'sick-561'}">
+      <!-- Theoretic FOV = 220 -->
+      <xacro:sick_tim561_laser name="${name}_laser" parent="${name}" ros_topic="scan_raw" update_rate="10" min_angle="${-110 * deg_to_rad}" max_angle="${110 * deg_to_rad}">
+        <origin xyz="${base_laser_x} ${base_laser_y} ${base_laser_z}" rpy="0 0 0" />
+      </xacro:sick_tim561_laser>
+    </xacro:if>
+    <!-- sick-571 -->
+    <xacro:if value="${laser_model == 'sick-571'}">
+      <!-- Theoretic FOV = 220 -->
+      <xacro:sick_tim571_laser name="${name}_laser" parent="${name}" ros_topic="scan_raw" update_rate="10" min_angle="${-110 * deg_to_rad}" max_angle="${110 * deg_to_rad}">
+        <origin xyz="${base_laser_x} ${base_laser_y} ${base_laser_z}" rpy="0 0 0" />
+      </xacro:sick_tim571_laser>
     </xacro:if>
     <!-- Sonars -->

Commit message: Change has_courier_rgbd_sensors to rgbd_sensors

File: pmb2_description/robots/pmb2.urdf.xacro (robot description, xacro)
@@ -21,5 +21,5 @@
   <xacro:arg name="has_microphone" default="false"/>
   <!-- false, true-->
-  <xacro:arg name="has_courier_rgbd_sensors" default="false"/>
+  <xacro:arg name="rgbd_sensors" default="false"/>
   <!-- Execution env config -->
   <xacro:arg name="use_sim_time" default="false"/>
@@ -32,5 +32,5 @@
   <xacro:property name="has_sonars" value="$(arg has_sonars)" />
   <xacro:property name="has_microphone" value="$(arg has_microphone)" />
-  <xacro:property name="has_courier_rgbd_sensors" value="$(arg has_courier_rgbd_sensors)"/>
+  <xacro:property name="rgbd_sensors" value="$(arg rgbd_sensors)"/>
   <!-- HW configuration check -->
   <xacro:if value="${laser_model not in ['no-laser', 'sick-551', 'sick-561', 'sick-571', 'hokuyo']}">
@@ -46,5 +46,5 @@
   <xacro:include filename="$(find pmb2_description)/urdf/base/base_sensors.urdf.xacro" />
   <!-- Courier rgbd sensors -->
-  <xacro:if value="${has_courier_rgbd_sensors}">
+  <xacro:if value="${rgbd_sensors}">
     <xacro:include filename="$(find pmb2_description)/urdf/cameras_add_on/cameras_add_on.urdf.xacro" />
   </xacro:if>
@@ -60,5 +60,5 @@
   <xacro:base_sensors name="base" laser_model="${laser_model}" has_sonars="${has_sonars}" has_microphone="${has_microphone}"/>
   <!-- RGBD Sensors -->
-  <xacro:if value="${has_courier_rgbd_sensors}">
+  <xacro:if value="${rgbd_sensors}">
     <xacro:cameras_add_on name="cameras_add_on" parent="base_link"/>
   </xacro:if>

Commit message: Change courier sensors to add-on-module

File: pmb2_description/robots/pmb2.urdf.xacro (robot description, xacro)
@@ -21,5 +21,5 @@
   <xacro:arg name="has_microphone" default="false"/>
   <!-- false, true-->
-  <xacro:arg name="rgbd_sensors" default="false"/>
+  <xacro:arg name="add_on_module" default="no-add-on"/>
   <!-- Execution env config -->
   <xacro:arg name="use_sim_time" default="false"/>
@@ -32,8 +32,11 @@
   <xacro:property name="has_sonars" value="$(arg has_sonars)" />
   <xacro:property name="has_microphone" value="$(arg has_microphone)" />
-  <xacro:property name="rgbd_sensors" value="$(arg rgbd_sensors)"/>
+  <xacro:property name="add_on_module" value="$(arg add_on_module)"/>
   <!-- HW configuration check -->
   <xacro:if value="${laser_model not in ['no-laser', 'sick-551', 'sick-561', 'sick-571', 'hokuyo']}">
     <xacro:wrong_laser_model/>
+  </xacro:if>
+  <xacro:if value="${add_on_module not in ['no-add-on', 'rgbd-sensors']}">
+    <xacro:wrong_add_on_module/>
   </xacro:if>
   <!-- Execution env configuration -->
@@ -46,5 +49,5 @@
   <xacro:include filename="$(find pmb2_description)/urdf/base/base_sensors.urdf.xacro" />
   <!-- Courier rgbd sensors -->
-  <xacro:if value="${rgbd_sensors}">
+  <xacro:if value="${add_on_module == 'rgbd-sensors'}">
     <xacro:include filename="$(find pmb2_description)/urdf/cameras_add_on/cameras_add_on.urdf.xacro" />
   </xacro:if>
@@ -60,5 +63,5 @@
   <xacro:base_sensors name="base" laser_model="${laser_model}" has_sonars="${has_sonars}" has_microphone="${has_microphone}"/>
   <!-- RGBD Sensors -->
-  <xacro:if value="${rgbd_sensors}">
+  <xacro:if value="${add_on_module == 'rgbd-sensors'}">
     <xacro:cameras_add_on name="cameras_add_on" parent="base_link"/>
   </xacro:if>

Commit message: add new gpu laser

File: pmb2_description/robots/pmb2.urdf.xacro (robot description, xacro)
@@ -15,5 +15,5 @@
   <!-- ARGUMENTS -->
   <!-- no-laser, hokuyo, sick-551, sick-561, sick-571-->
-  <xacro:arg name="laser_model" default="sick-571"/>
+  <xacro:arg name="laser_model" default="sick-571-gpu"/>
   <!-- false, true -->
   <xacro:arg name="has_sonars" default="true"/>
@@ -34,5 +34,5 @@
   <xacro:property name="add_on_module" value="$(arg add_on_module)"/>
   <!-- HW configuration check -->
-  <xacro:if value="${laser_model not in ['no-laser', 'sick-551', 'sick-561', 'sick-571', 'hokuyo']}">
+  <xacro:if value="${laser_model not in ['no-laser', 'sick-551', 'sick-561', 'sick-571', 'sick-571-gpu', 'hokuyo']}">
     <xacro:wrong_laser_model/>
   </xacro:if>

File: pmb2_description/urdf/base/base_sensors.urdf.xacro (robot description, xacro)
@@ -24,4 +24,5 @@
   <xacro:include filename="$(find pmb2_description)/urdf/sensors/sick_tim561_laser.urdf.xacro"/>
   <xacro:include filename="$(find pmb2_description)/urdf/sensors/sick_tim571_laser.urdf.xacro"/>
+  <xacro:include filename="$(find pmb2_description)/urdf/sensors/sick_tim571_laser_gpu.urdf.xacro"/>
   <xacro:include filename="$(find pmb2_description)/urdf/sensors/range.urdf.xacro"/>
   <xacro:include filename="$(find pmb2_description)/urdf/sensors/microphone.urdf.xacro"/>
@@ -61,4 +62,11 @@
       </xacro:sick_tim571_laser>
     </xacro:if>
+    <!-- sick-571-gpu -->
+    <xacro:if value="${laser_model == 'sick-571-gpu'}">
+      <!-- Theoretic FOV = 220 -->
+      <xacro:sick_tim571_laser_gpu name="${name}_laser" parent="${name}_link" ros_topic="scan_raw" update_rate="10" min_angle="${-110 * deg_to_rad}" max_angle="${110 * deg_to_rad}">
+        <origin xyz="${base_laser_x} ${base_laser_y} ${base_laser_z}" rpy="0 0 0" />
+      </xacro:sick_tim571_laser_gpu>
+    </xacro:if>
     <!-- Sonars -->
     <xacro:if value="${has_sonars}">
